Commit message: Changed a lot of things

File: exo_description/urdf/lleap_exo.urdf.xacro (robot description, xacro)
@@ -29,6 +29,9 @@
         the world frame (the ground plane), you must create a "world"
         link and a joint that fixes it to the base of your model." -->
+ <!--
   <link name="world"/>
+-->
   <!-- secure (fix) model in Gazebo: world <> link0 = fixed base_link = torso -->
+  <!--
   <joint name="global_fixed" type="fixed">
     <origin xyz="0 0 1" rpy="0 0 ${pi}" />
@@ -36,4 +39,5 @@
     <child link="base_link"/>
   </joint>
+-->
   <!-- torso: base for the model; attached to world in gazebo if whole model fixed -->
   <link name="base_link">
@@ -100,4 +104,5 @@
       <!-- Positional joint limits partially based on Tamar's msts (upper lim here). -->
       <limit lower="${hip_lower_radians}" upper="${hip_upper_radians}" effort="700" velocity="5" />
+      <dynamics damping="1.0" friction="0.05" spring_stiffness="250" spring_reference="0"/>
     </joint>
     <!-- link1 should be the thigh (joint1 to joint2).
@@ -135,4 +140,5 @@
       <!-- Positional joint limits partially based on Tamar's msts (lower lim here). -->
       <limit lower="${knee_lower_radians}" upper="${knee_upper_radians}" effort="250" velocity="1.308" />
+      <dynamics damping="1.0" friction="0.05" spring_stiffness="250" spring_reference="0"/>
     </joint>
     <!-- link2 should be the shank (joint2 to joint3).
@@ -171,10 +177,9 @@
       <!-- Positional joint limits NOT based on Tamar's msts, but normal ranges instead. -->
       <limit lower="${ankle_lower_radians}" upper="${ankle_upper_radians}" effort="250" velocity="1.308" />
+      <dynamics damping="1.0" friction="0.05" spring_stiffness="250" spring_reference="0"/>
     </joint>
     <!-- link3 should be the foot. -->
     <link name="${prefix}_${link3}">
       <inertial>
-        <!-- TODO: probably need to change this interial element -->
-        <!-- not quite sure what this is <origin xyz="-0.210873385399549 -0.0276710830621445 -0.140982468689507" rpy="0 0 0" /> -->
         <mass value="1.10275445439595" />
         <inertia ixx="0.00199044634689737" ixy="-7.54331572697175E-06" ixz="-0.00260077424938593" iyy="0.00581565190920448" iyz="-4.96554466328964E-06" izz="0.00412555905043524" />
@@ -219,18 +224,2 @@
   -->
 </robot>
-<!--
-  TODO: consider reorganizing a bit to be more modularly structured like the UR robot arm URDFs.
-  Don't need to be as modular bc only one robot (i.e., not ur3, ur5, etc) and less complex so far,
-    but good to keep some things in mind as reference -> potential future changes to our model.
-  - transmissions in separate file; macro for one leg's transmissions, prefix (usual) and
-      hw_interface as marco params
-  - see the xacro:insert_clock use in the _robot. files
-    https://answers.ros.org/question/358472/xacro-insert_block-parameter/
-    any use for us?
-  - also see creation and use of the xacro macro cylinder intertial.
-    if we build our simple geom model as cylinders (looking like the UR arms tbh), can use something
-      similar to calc/create inertial blocks?
-  - overall, just note which components (basic links and joints, transmissions, other gazebo
-    components like intertials and plugins, macros, properties, etc)
-  https://github.com/ros-industrial/universal_robot/blob/melodic-devel/ur_description/urdf/ur3.urdf.xacro
--->

File: exo_description/urdf/lleap_exo_gazebo.xacro (robot description, xacro)
@@ -30,3 +30,31 @@
     </plugin>
   </gazebo>
+  <!-- Adding IMU sensor plugin to the base_link -->
+  <gazebo reference="base_link">
+    <sensor type="imu" name="imu_sensor">
+      <always_on>true</always_on>
+      <update_rate>50</update_rate>
+      <imu>
+        <angular_velocity>
+          <noise type="gaussian">
+            <mean>0.0</mean>
+            <stddev>0.01</stddev>
+          </noise>
+        </angular_velocity>
+        <linear_acceleration>
+          <noise type="gaussian">
+            <mean>0.0</mean>
+            <stddev>0.01</stddev>
+          </noise>
+        </linear_acceleration>
+      </imu>
+      <plugin name="imu_sensor" filename="libgazebo_ros_imu_sensor.so">
+        <ros>
+          <namespace>imu</namespace>
+          <remapping>~/out:=data</remapping>
+        </ros>
+        <initial_orientation_as_reference>false</initial_orientation_as_reference>
+      </plugin>
+    </sensor>
+  </gazebo>
 </robot>

File: exo_moveit/config/lleap_exo.urdf.xacro (robot description, xacro)
@@ -6,4 +6,5 @@
     <!-- Import control_xacro -->
     <xacro:include filename="lleap_exo.ros2_control.xacro" />
+    <xacro:include filename="transmissions.xacro" />
     <xacro:lleap_exo_ros2_control name="FakeSystem" initial_positions_file="$(arg initial_positions_file)"/>
 </robot>

Commit message: So much code later

File: exo_description/urdf/lleap_exo.urdf.xacro (robot description, xacro)
@@ -1,3 +1,3 @@
-<?xml version="1.0" encoding="utf-8" ?>
+<?xml version="1.1" encoding="utf-8" ?>
 <!-- This URDF was automatically created by SolidWorks to URDF Exporter! Originally created by Stephen Brawner (brawner@gmail.com)
      Commit Version: 1.6.0-1-g15f4949  Build Version: 1.6.7594.29634
@@ -8,7 +8,15 @@
     the namespace (in gazebo plugin at the bottom) to match. -->
   <xacro:property name="robot_name" value="exo" />
+  <xacro:arg name="use_fake_hardware" default="false"/>
+  <xacro:property name="_fake" value="$(arg use_fake_hardware)" />
   <!-- Grab the joint limits. -->
   <xacro:include filename="$(find exo_description)/urdf/lleap_exo_joint_limits.xacro" />
   <xacro:include filename="$(find exo_description)/urdf/exo_material_colors.xacro"/>
+  <xacro:if value="${_fake}">
+    <xacro:include filename="$(find exo_description)/urdf/lleap_exo.ros2_control.fake.xacro"/>
+  </xacro:if>
+  <xacro:unless value="${_fake}">
+    <xacro:include filename="$(find exo_description)/urdf/lleap_exo.ros2_control.xacro"/>
+  </xacro:unless>
   <!-- link names; 1-3 map to .STL filenames -->
   <xacro:property name="link0" value="hip_base" />  <!-- stationary inner part of hip joint -->
@@ -29,11 +37,11 @@
         the world frame (the ground plane), you must create a "world"
         link and a joint that fixes it to the base of your model." -->
-  <link name="world"/>
+  <!-- <link name="world"/> -->
   <!-- secure (fix) model in Gazebo: world <> link0 = fixed base_link = torso -->
-  <joint name="global_fixed" type="fixed">
+  <!-- <joint name="global_fixed" type="fixed">
     <origin xyz="0 0 1" rpy="0 0 ${pi}" />
     <parent link="world"/>
     <child link="base_link"/>
-  </joint>
+  </joint> -->
   <!-- torso: base for the model; attached to world in gazebo if whole model fixed -->
   <link name="base_link">
@@ -41,5 +49,5 @@
       <origin xyz="0 0 0.5" rpy="0 0 0" />
       <!-- TODO: don't forget to add torso mass (and whole intertial element) here once have an estimate! -->
-      <mass value="0" />
+      <mass value="30" />
       <geometry>
         <box size="0.25 ${torso_width} 1"/>
@@ -198,5 +206,5 @@
   <xacro:leg prefix="right" reflect="1" />
   <xacro:leg prefix="left" reflect="-1" />
-  <xacro:include filename="$(find exo_description)/urdf/lleap_exo_gazebo.xacro" />
+  <!-- <xacro:include filename="$(find exo_description)/urdf/lleap_exo_gazebo.xacro" /> -->
   <!-- Needed gazebo_ros_control plugin.
   <gazebo>

File: exo_description/urdf/lleap_exo_gazebo.xacro (robot description, xacro)
@@ -1,5 +1,4 @@
 <?xml version="1.0" encoding='utf-8' ?>
 <robot xmlns:xacro="http://www.ros.org/wiki/xacro">
-  <!-- Gazebo requires the use of plugins to interact with other systems such as ROS. -->
   <!-- This plugin will publish the joint_states for the selected joints
           (which robot_state_publisher can then use to broadcast the approprate tf). -->

Commit message: Add gazebo fortress

File: exo_description/urdf/lleap_exo.urdf.xacro (robot description, xacro)
@@ -9,5 +9,7 @@
   <xacro:property name="robot_name" value="exo" />
   <xacro:arg name="use_fake_hardware" default="false"/>
+  <xacro:arg name="use_gazebo_fortress" default="false"/>
   <xacro:property name="_fake" value="$(arg use_fake_hardware)" />
+  <xacro:property name="_fortress" value="$(arg use_gazebo_fortress)" />
   <!-- Grab the joint limits. -->
   <xacro:include filename="$(find exo_description)/urdf/lleap_exo_joint_limits.xacro" />
@@ -46,8 +48,11 @@
   <!-- torso: base for the model; attached to world in gazebo if whole model fixed -->
   <link name="base_link">
+    <inertial>
+      <origin xyz="0 0 0.5" rpy="0 0 0" />
+      <mass value="30" />
+      <inertia ixx="2.5625" ixy="0.0" ixz="0.0" iyy="2.6042" iyz="0.0" izz="0.1562" />
+    </inertial>
     <visual>
       <origin xyz="0 0 0.5" rpy="0 0 0" />
-      <!-- TODO: don't forget to add torso mass (and whole intertial element) here once have an estimate! -->
-      <mass value="30" />
       <geometry>
         <box size="0.25 ${torso_width} 1"/>
@@ -55,4 +60,10 @@
       <material name="red"/>
     </visual>
+    <collision>
+      <origin xyz="0 0 0.5" rpy="0 0 0" />
+      <geometry>
+        <box size="0.25 ${torso_width} 1"/>
+      </geometry>
+    </collision>
   </link>
   <!-- xacro macro for a leg (including Gazebo transmission elements).
@@ -206,5 +217,13 @@
   <xacro:leg prefix="right" reflect="1" />
   <xacro:leg prefix="left" reflect="-1" />
-  <!-- <xacro:include filename="$(find exo_description)/urdf/lleap_exo_gazebo.xacro" /> -->
+  <!-- Include Gazebo plugins based on which simulator is being used -->
+  <xacro:if value="${_fortress}">
+    <!-- Gazebo Fortress/Ignition plugins -->
+    <xacro:include filename="$(find exo_description)/urdf/lleap_exo_gazebo_fortress.xacro" />
+  </xacro:if>
+  <xacro:unless value="${_fortress}">
+    <!-- Gazebo Classic plugins -->
+    <xacro:include filename="$(find exo_description)/urdf/lleap_exo_gazebo.xacro" />
+  </xacro:unless>
   <!-- Needed gazebo_ros_control plugin.
   <gazebo>
